File: PCB/MosfetBase/mosfetModule.kicad_pcb (KiCad board)
At the start: 2 copper layers, 75.5 x 45.5 mm, 29 parts, among them J1 toDCCnext, J2 power, J3 point, J4 point, J5 point, J6 point, SW1 SW_SPST, U1 IRF71xx, U2 IRF71xx, U3 IRF71xx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

Commit message: added signal base, fixed vias on mosgfet modules
Routing:
- net Net-(A1-Pad5): vias 1 -> 0
- net Net-(A1-Pad14): vias 1 -> 0
- net GND: vias 51 -> 56
- net /in3-2: vias 2 -> 1
- net /in3-1: vias 1 -> 0
- net /in2-1: vias 1 -> 0
