File: PCB/base_modules/SignalBase/dccSignals.sch (KiCad schematic (older format))
At the start: 13 parts, among them J1 Screw_Terminal_01x02, J3 leds, J4 leds, J5 leds, J6 leds, SW1 SW_SPST, U1 ULN2003A, U2 ULN2003A, U3 ATmega328-PU

Commit message: routed signals PCB.
Was thinking to make a loconet block unit. Combined feedback, as well as
signal and ABC module. This would allow for automatic analog block
system for digital trains.
Also was thinking to make 2 separate blocks on 1 one pcb, provided if possible
Parts:
- removed A2: Arduino_Nano_v2.x, Module:Arduino_Nano, symbol MCU_Module:Arduino_Nano_v2.x
- removed U3: ATmega328-PU, Package_DIP:DIP-28_W7.62mm, symbol MCU_Microchip_ATmega:ATmega328-PU
Connections:
- net VCC: no longer U1.9 (COM), U2.9 (COM)
- no-connect marks 18 -> 20
Changed lines of the file:
@@
 Text Label 2200 4300 2    50   ~ 0
 S1R_IN
-Wire Wire Line
-	7300 2650 7600 2650
-Wire Wire Line
-	7300 1000 7600 1000
 $Comp
 L MCU_Module:Arduino_Nano_v2.x A1
@@
 $EndComp
 $Comp
-L power:VCC #PWR0110
-U 1 1 62518E49
-P 7600 2300
-F 0 "#PWR0110" H 7600 2150 50  0001 C CNN
-F 1 "VCC" H 7615 2473 50  0000 C CNN
-F 2 "" H 7600 2300 50  0001 C CNN
-F 3 "" H 7600 2300 50  0001 C CNN
-	1    7600 2300
-	1    0    0    -1
-$EndComp
-Wire Wire Line
-	7600 2300 7600 2650
-$Comp
-L power:VCC #PWR0111
-U 1 1 62518A5A
-P 7600 900
-F 0 "#PWR0111" H 7600 750 50  0001 C CNN
-F 1 "VCC" H 7615 1073 50  0000 C CNN
-F 2 "" H 7600 900 50  0001 C CNN
-F 3 "" H 7600 900 50  0001 C CNN
-	1    7600 900
-	1    0    0    -1
-$EndComp
-$Comp
 L Transistor_Array:ULN2003A U1
 U 1 1 62524260
@@
 	1    0    0    -1
 $EndComp
-Wire Wire Line
-	7600 1000 7600 900
 $Comp
 L Transistor_Array:ULN2003A U2
@@
 Wire Wire Line
 	2750 2450 2950 2450
-$Comp
-L MCU_Module:Arduino_Nano_v2.x A2
-U 1 1 626EEC29
-P 8450 5400
-F 0 "A2" H 7900 4400 50  0000 C CNN
-F 1 "Arduino_Nano_v2.x" H 7850 4300 50  0000 C CNN
-F 2 "Module:Arduino_Nano" H 8450 5400 50  0001 C CIN
-F 3 "https://www.arduino.cc/en/uploads/Main/ArduinoNanoManual23.pdf" H 8450 5400 50  0001 C CNN
-	1    8450 5400
-	1    0    0    -1
-$EndComp
-$Comp
-L MCU_Microchip_ATmega:ATmega328-PU U3
-U 1 1 626F37B4
-P 10350 5550
-F 0 "U3" H 9706 5596 50  0000 R CNN
-F 1 "ATmega328-PU" H 9706 5505 50  0000 R CNN
-F 2 "Package_DIP:DIP-28_W7.62mm" H 10350 5550 50  0001 C CIN
-F 3 "http://ww1.microchip.com/downloads/en/DeviceDoc/ATmega328_P%20AVR%20MCU%20with%20picoPower%20Technology%20Data%20Sheet%2040001984A.pdf" H 10350 5550 50  0001 C CNN
-	1    10350 5550
-	1    0    0    -1
-$EndComp
+NoConn ~ 7300 1000
+NoConn ~ 7300 2650
 $EndSCHEMATC
