File: PCB/ServoBase/ServoBase.kicad_pcb (KiCad board)
At the start: 2 copper layers, 55 x 60 mm, 30 parts, among them J1 servo, J2 servo, J3 servo, J4 servo, J6 frog, J7 DCC, J8 frog, J9 pow, K1 G5V-1, K2 G5V-1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

Commit message: many changes made..
Parts:
- added R2: R, Resistor_THT:R_Axial_DIN0204_L3.6mm_D1.6mm_P7.62mm_Horizontal, F.Cu at (135.6, 80.0)
Connections:
- A1 pad 14: /conf -> Net-(A1-Pad14)
- A1 pad 25: Net-(A1-Pad25) -> /conf
Routing:
- net +5V: track 0.00 -> 138.8 mm
- net /DCC+: track 0.00 -> 68.1 mm
- net /DCC-: track 0.00 -> 64.2 mm
- net /mot4: track 0.00 -> 59.3 mm
- net /mot3: track 0.00 -> 53.6 mm
- net Net-(C1-Pad1): track 0.00 -> 52.4 mm
- net /mot2: track 0.00 -> 49.1 mm
- net /mot1: track 0.00 -> 45.2 mm
- net /pot1: track 0.00 -> 42.1 mm
- net /pot2: track 0.00 -> 41.8 mm
- net /conf: track 0.00 -> 32.5 mm
- net Net-(D2-Pad2): track 0.00 -> 26.1 mm
- net /status: track 0.00 -> 25.9 mm
- net /coil4: track 0.00 -> 24.5 mm
- net /coil1: track 0.00 -> 23.5 mm
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- added copper zone on B.Cu, net GND
- added copper zone on F.Cu, net GND
Other:
- board text added: "12v - gnd"
- board text added: "Servo Base w/ Frog By Bas Knippels"
