File: PCB/ServoBase/ServoBase.sch (KiCad schematic (older format))
At the start: 27 parts, among them J1 servo, J2 servo, J3 servo, J4 servo, J5 Btn, J6 frog, J7 DCC, J8 frog, J9 pow, K1 G5V-1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

Commit message: many changes made..
Parts:
- added R2: R, Resistor_THT:R_Axial_DIN0204_L3.6mm_D1.6mm_P7.62mm_Horizontal, symbol Device:R
Connections:
- net +5V: now also R2.1
- net conf: now also A1.25 (A6), R2.2; no longer A1.14 (D11)
Other:
- moved on the sheet: SW1
Changed lines of the file:
@@
 L Switch:SW_SPST SW1
 U 1 1 6239B121
-P 2850 4950
-F 0 "SW1" H 2850 5185 50  0000 C CNN
-F 1 "conf" H 2850 5094 50  0000 C CNN
-F 2 "Button_Switch_THT:SW_PUSH_6mm_H4.3mm" H 2850 4950 50  0001 C CNN
-F 3 "~" H 2850 4950 50  0001 C CNN
-	1    2850 4950
+P 2950 4950
+F 0 "SW1" H 2950 5185 50  0000 C CNN
+F 1 "conf" H 2950 5094 50  0000 C CNN
+F 2 "Button_Switch_THT:SW_PUSH_6mm_H4.3mm" H 2950 4950 50  0001 C CNN
+F 3 "~" H 2950 4950 50  0001 C CNN
+	1    2950 4950
 	1    0    0    -1
 $EndComp
@@
 L power:GND #PWR0124
 U 1 1 6239E685
-P 2600 4950
-F 0 "#PWR0124" H 2600 4700 50  0001 C CNN
-F 1 "GND" H 2605 4777 50  0000 C CNN
-F 2 "" H 2600 4950 50  0001 C CNN
-F 3 "" H 2600 4950 50  0001 C CNN
-	1    2600 4950
-	1    0    0    -1
-$EndComp
-Wire Wire Line
-	2600 4950 2650 4950
-Wire Wire Line
-	3050 4950 3200 4950
-Text Label 3200 4950 2    50   ~ 0
+P 2700 4950
+F 0 "#PWR0124" H 2700 4700 50  0001 C CNN
+F 1 "GND" H 2705 4777 50  0000 C CNN
+F 2 "" H 2700 4950 50  0001 C CNN
+F 3 "" H 2700 4950 50  0001 C CNN
+	1    2700 4950
+	1    0    0    -1
+$EndComp
+Wire Wire Line
+	2700 4950 2750 4950
+Text Label 3400 4950 2    50   ~ 0
 conf
-Text Label 4250 3850 0    50   ~ 0
-conf
-Wire Wire Line
-	4250 3850 4550 3850
 $Comp
 L power:GND #PWR0125
@@
 	5550 3750 5800 3750
 NoConn ~ 5550 4050
-NoConn ~ 5550 3950
 Text Label 5800 3850 2    50   ~ 0
 pot2
@@
 Wire Wire Line
 	2950 1050 2950 1350
+Text Label 5800 3950 2    50   ~ 0
+conf
+Wire Wire Line
+	5550 3950 5800 3950
+NoConn ~ 4550 3850
+$Comp
+L Device:R R2
+U 1 1 623B6C99
+P 3400 4750
+F 0 "R2" V 3193 4750 50  0000 C CNN
+F 1 "R" V 3284 4750 50  0000 C CNN
+F 2 "Resistor_THT:R_Axial_DIN0204_L3.6mm_D1.6mm_P7.62mm_Horizontal" V 3330 4750 50  0001 C CNN
+F 3 "~" H 3400 4750 50  0001 C CNN
+	1    3400 4750
+	0    1    1    0
+$EndComp
+Wire Wire Line
+	3150 4950 3200 4950
+Wire Wire Line
+	3250 4750 3200 4750
+Wire Wire Line
+	3200 4750 3200 4950
+Connection ~ 3200 4950
+Wire Wire Line
+	3200 4950 3400 4950
+$Comp
+L power:+5V #PWR0130
+U 1 1 623BEFA7
+P 3650 4750
+F 0 "#PWR0130" H 3650 4600 50  0001 C CNN
+F 1 "+5V" H 3665 4923 50  0000 C CNN
+F 2 "" H 3650 4750 50  0001 C CNN
+F 3 "" H 3650 4750 50  0001 C CNN
+	1    3650 4750
+	1    0    0    -1
+$EndComp
+Wire Wire Line
+	3650 4750 3550 4750
 $EndSCHEMATC
