File: PCB/base_modules/controlPanelBase/switchController.kicad_pcb (KiCad board)
At the start: 2 copper layers, 61.5 x 40 mm, 15 parts, among them J1 i, J10 i, J2 i, J3 i, J4 i, J7 i, J8 i, J9 i, SW1 SW_SPST

Commit message: added gerber files in the release folder for all base units. The interfaces are not yet done
Other:
- board text added: "Control panel base By Bas Knippels"
- board text removed: "Switch panel module By Bas Knippels"
- board text removed: "switchController V1.0 By Bas Knippels"
